File: kicad/frontend.kicad_sch (KiCad schematic)
At the start: 0 parts

Commit message: I dont remember last commit idk
Parts:
- added C1, C8: 0.1u, symbol Device:C
- added R17, R18, R20: 10k, symbol Device:R
- added R19, R21: 20k, symbol Device:R
Connections:
- net 3v3: now also C8.1, R18.1, R21.1
- new net ANALOG_IN: C1.2
- new net GND: C8.2, R17.2, R19.2
- new net OPA_N: R19.1, R20.1, R21.2
- new net OPA_OUT: R20.2
- new net OPA_P: C1.1, R17.1, R18.2
